Commit message: Fixed sensor bug in nexus sim

File: nexus_4wd_mecanum_description/urdf/nexus_4wd_mecanum.xacro (robot description, xacro)
@@ -273,7 +273,7 @@
     <origin xyz="0 0.108 0.010" rpy="0 0 ${PI/2}" />
     <parent link="base_link"/>
-    <child link="left_sensor" />
-  </joint>
-  <link name="left_sensor">
+    <child link="left_range" />
+  </joint>
+  <link name="left_range">
     <visual>
       <origin xyz="0 0 0" rpy="${PI/2} 0 0" />
@@ -287,7 +287,7 @@
     <origin xyz="0.205 0 0.010" rpy="0 0 0" />
     <parent link="base_link"/>
-    <child link="front_sensor" />
-  </joint>
-  <link name="front_sensor">
+    <child link="front_range" />
+  </joint>
+  <link name="front_range">
     <visual>
       <origin xyz="0 0 0" rpy="${PI/2} 0 0" />
@@ -301,7 +301,7 @@
     <origin xyz="0 -0.108 0.010" rpy="0 0 ${-PI/2}" />
     <parent link="base_link"/>
-    <child link="right_sensor" />
-  </joint>
-  <link name="right_sensor">
+    <child link="right_range" />
+  </joint>
+  <link name="right_range">
     <visual>
       <origin xyz="0 0 0" rpy="${PI/2} 0 0" />
@@ -315,7 +315,7 @@
     <origin xyz="-0.201 0 0.010" rpy="0 0 ${PI}" />
     <parent link="base_link"/>
-    <child link="rear_sensor" />
-  </joint>
-  <link name="rear_sensor">
+    <child link="rear_range" />
+  </joint>
+  <link name="rear_range">
     <visual>
       <origin xyz="0 0 0" rpy="${PI/2} 0 0" />
@@ -331,10 +331,10 @@
   <xacro:include filename="$(find nexus_4wd_mecanum_description)/urdf/urm04_sensor.xacro"/>
   <!-- front sensor -->
-  <xacro:urm04_sensor frame_name="front_range" ros_topic="front_sensor" update_rate="10" min_range="0.04" max_range="2.5" horizontal_field_of_view="1.04" vertical_field_of_view="0.04" ray_count="2" />
+  <xacro:urm04_sensor frame_name="front_range" ros_topic="front_range" update_rate="10" min_range="0.01" max_range="2.5" horizontal_field_of_view="1.57" vertical_field_of_view="0.1" ray_count="2" />
   <!-- left sensor -->
-  <xacro:urm04_sensor frame_name="left_range" ros_topic="left_sensor" update_rate="10" min_range="0.04" max_range="2.5" horizontal_field_of_view="1.04" vertical_field_of_view="0.04" ray_count="2" />
+  <xacro:urm04_sensor frame_name="left_range" ros_topic="left_range" update_rate="10" min_range="0.01" max_range="2.5" horizontal_field_of_view="1.57" vertical_field_of_view="0.1" ray_count="2" />
   <!-- right sensor -->
-  <xacro:urm04_sensor frame_name="right_range" ros_topic="right_sensor" update_rate="10" min_range="0.04" max_range="2.5" horizontal_field_of_view="1.04" vertical_field_of_view="0.04" ray_count="2" />
+  <xacro:urm04_sensor frame_name="right_range" ros_topic="right_range" update_rate="10" min_range="0.01" max_range="2.5" horizontal_field_of_view="1.57" vertical_field_of_view="0.1" ray_count="2" />
   <!-- rear sensor -->
-  <xacro:urm04_sensor frame_name="rear_range" ros_topic="rear_sensor" update_rate="10" min_range="0.04" max_range="2.5" horizontal_field_of_view="1.04" vertical_field_of_view="0.04" ray_count="2" />
+  <xacro:urm04_sensor frame_name="rear_range" ros_topic="rear_range" update_rate="10" min_range="0.01" max_range="2.5" horizontal_field_of_view="1.57" vertical_field_of_view="0.1" ray_count="2" />
 </robot>

File: nexus_4wd_mecanum_description/urdf/urm04_sensor.xacro (robot description, xacro)
@@ -29,11 +29,10 @@
         </ray>
         <plugin name="gazebo_ros_${frame_name}" filename="libgazebo_ros_range.so">
-          <always_on>true</always_on>
-          <update_rate>${update_rate}</update_rate>
+          <updateRate>${update_rate}</updateRate>
           <gaussianNoise>0.005</gaussianNoise>
           <topicName>${ros_topic}</topicName>
-          <frameId>${frame_name}</frameId>
+          <frameName>${frame_name}</frameName>
           <radiation>INFRARED</radiation>
-          <fov>0.2967</fov>
+          <fov>1.57</fov>
         </plugin>
       </sensor>

Commit message: Modified sensor positioning s.t. sensing cone doesn't intercept ground

File: nexus_4wd_mecanum_description/urdf/nexus_4wd_mecanum.xacro (robot description, xacro)
@@ -271,5 +271,5 @@
   </link>
   <joint name="left_sensor_joint" type="fixed">
-    <origin xyz="0 0.108 0.010" rpy="0 0 ${PI/2}" />
+    <origin xyz="0 0.108 0.010" rpy="0 -0.1 ${PI/2}" />
     <parent link="base_link"/>
     <child link="left_range" />
@@ -285,5 +285,5 @@
   </link>
   <joint name="front_sensor_joint" type="fixed">
-    <origin xyz="0.205 0 0.010" rpy="0 0 0" />
+    <origin xyz="0.205 0 0.010" rpy="0 -0.1 0" />
     <parent link="base_link"/>
     <child link="front_range" />
@@ -299,5 +299,5 @@
   </link>
   <joint name="right_sensor_joint" type="fixed">
-    <origin xyz="0 -0.108 0.010" rpy="0 0 ${-PI/2}" />
+    <origin xyz="0 -0.108 0.010" rpy="0 -0.1 ${-PI/2}" />
     <parent link="base_link"/>
     <child link="right_range" />
@@ -313,5 +313,5 @@
   </link>
   <joint name="rear_sensor_joint" type="fixed">
-    <origin xyz="-0.201 0 0.010" rpy="0 0 ${PI}" />
+    <origin xyz="-0.201 0 0.010" rpy="0 -0.1 ${PI}" />
     <parent link="base_link"/>
     <child link="rear_range" />
@@ -331,10 +331,10 @@
   <xacro:include filename="$(find nexus_4wd_mecanum_description)/urdf/urm04_sensor.xacro"/>
   <!-- front sensor -->
-  <xacro:urm04_sensor frame_name="front_range" ros_topic="front_range" update_rate="10" min_range="0.01" max_range="2.5" horizontal_field_of_view="1.57" vertical_field_of_view="0.1" ray_count="2" />
+  <xacro:urm04_sensor frame_name="front_range" ros_topic="front_range" update_rate="10" min_range="0.01" max_range="2" horizontal_field_of_view="0.261799" vertical_field_of_view="0.2" ray_count="2" />
   <!-- left sensor -->
-  <xacro:urm04_sensor frame_name="left_range" ros_topic="left_range" update_rate="10" min_range="0.01" max_range="2.5" horizontal_field_of_view="1.57" vertical_field_of_view="0.1" ray_count="2" />
+  <xacro:urm04_sensor frame_name="left_range" ros_topic="left_range" update_rate="10" min_range="0.01" max_range="2" horizontal_field_of_view="0.261799" vertical_field_of_view="0.2" ray_count="2" />
   <!-- right sensor -->
-  <xacro:urm04_sensor frame_name="right_range" ros_topic="right_range" update_rate="10" min_range="0.01" max_range="2.5" horizontal_field_of_view="1.57" vertical_field_of_view="0.1" ray_count="2" />
+  <xacro:urm04_sensor frame_name="right_range" ros_topic="right_range" update_rate="10" min_range="0.01" max_range="2" horizontal_field_of_view="0.261799" vertical_field_of_view="0.2" ray_count="2" />
   <!-- rear sensor -->
-  <xacro:urm04_sensor frame_name="rear_range" ros_topic="rear_range" update_rate="10" min_range="0.01" max_range="2.5" horizontal_field_of_view="1.57" vertical_field_of_view="0.1" ray_count="2" />
+  <xacro:urm04_sensor frame_name="rear_range" ros_topic="rear_range" update_rate="10" min_range="0.01" max_range="2" horizontal_field_of_view="0.261799" vertical_field_of_view="0.2" ray_count="2" />
 </robot>

File: nexus_4wd_mecanum_description/urdf/urm04_sensor.xacro (robot description, xacro)
@@ -34,5 +34,5 @@
           <frameName>${frame_name}</frameName>
           <radiation>INFRARED</radiation>
-          <fov>1.57</fov>
+          <fov>${horizontal_field_of_view/2}</fov>
         </plugin>
       </sensor>

Commit message: Added support for 8 ToF sensors on robot

File: nexus_4wd_mecanum_description/urdf/nexus_4wd_mecanum.xacro (robot description, xacro)
@@ -326,4 +326,60 @@
     </visual>
   </link>
+  <joint name="front_right_sensor_joint" type="fixed">
+    <origin xyz="0.201 -0.108 0.010" rpy="0 -0.1 ${-PI/4}" />
+    <parent link="base_link"/>
+    <child link="front_right_range" />
+  </joint>
+  <link name="front_right_range">
+    <visual>
+      <origin xyz="0 0 0" rpy="${PI/2} 0 0" />
+      <geometry>
+        <mesh filename="package://nexus_4wd_mecanum_description/meshes/urm04.STL" scale="0.001 0.001 0.001"/>
+      </geometry>
+      <material name="black" />
+    </visual>
+  </link>
+  <joint name="front_left_sensor_joint" type="fixed">
+    <origin xyz="0.201 0.108 0.010" rpy="0 -0.1 ${PI/4}" />
+    <parent link="base_link"/>
+    <child link="front_left_range" />
+  </joint>
+  <link name="front_left_range">
+    <visual>
+      <origin xyz="0 0 0" rpy="${PI/2} 0 0" />
+      <geometry>
+        <mesh filename="package://nexus_4wd_mecanum_description/meshes/urm04.STL" scale="0.001 0.001 0.001"/>
+      </geometry>
+      <material name="black" />
+    </visual>
+  </link>
+  <joint name="rear_right_sensor_joint" type="fixed">
+    <origin xyz="-0.201 -0.108 0.010" rpy="0 -0.1 ${-3*PI/4}" />
+    <parent link="base_link"/>
+    <child link="rear_right_range" />
+  </joint>
+  <link name="rear_right_range">
+    <visual>
+      <origin xyz="0 0 0" rpy="${PI/2} 0 0" />
+      <geometry>
+        <mesh filename="package://nexus_4wd_mecanum_description/meshes/urm04.STL" scale="0.001 0.001 0.001"/>
+      </geometry>
+      <material name="black" />
+    </visual>
+  </link>
+  <joint name="rear_left_sensor_joint" type="fixed">
+    <origin xyz="-0.201 0.108 0.010" rpy="0 -0.1 ${3*PI/4}" />
+    <parent link="base_link"/>
+    <child link="rear_left_range" />
+  </joint>
+  <link name="rear_left_range">
+    <visual>
+      <origin xyz="0 0 0" rpy="${PI/2} 0 0" />
+      <geometry>
+        <mesh filename="package://nexus_4wd_mecanum_description/meshes/urm04.STL" scale="0.001 0.001 0.001"/>
+      </geometry>
+      <material name="black" />
+    </visual>
+  </link>
   <!-- Include controller plugin for Gazebo -->
   <xacro:include filename="$(find nexus_4wd_mecanum_description)/urdf/nexus_4wd_mecanum.gazebo" />
@@ -331,10 +387,14 @@
   <xacro:include filename="$(find nexus_4wd_mecanum_description)/urdf/urm04_sensor.xacro"/>
   <!-- front sensor -->
-  <xacro:urm04_sensor frame_name="front_range" ros_topic="front_range" update_rate="10" min_range="0.01" max_range="2" horizontal_field_of_view="0.261799" vertical_field_of_view="0.2" ray_count="2" />
+  <xacro:urm04_sensor frame_name="front_range" ros_topic="front_range" update_rate="10" min_range="0.01" max_range="2" horizontal_field_of_view="0.261799" vertical_field_of_view="0.2" ray_count="5" />
   <!-- left sensor -->
-  <xacro:urm04_sensor frame_name="left_range" ros_topic="left_range" update_rate="10" min_range="0.01" max_range="2" horizontal_field_of_view="0.261799" vertical_field_of_view="0.2" ray_count="2" />
+  <xacro:urm04_sensor frame_name="left_range" ros_topic="left_range" update_rate="10" min_range="0.01" max_range="2" horizontal_field_of_view="0.261799" vertical_field_of_view="0.2" ray_count="5" />
   <!-- right sensor -->
-  <xacro:urm04_sensor frame_name="right_range" ros_topic="right_range" update_rate="10" min_range="0.01" max_range="2" horizontal_field_of_view="0.261799" vertical_field_of_view="0.2" ray_count="2" />
+  <xacro:urm04_sensor frame_name="right_range" ros_topic="right_range" update_rate="10" min_range="0.01" max_range="2" horizontal_field_of_view="0.261799" vertical_field_of_view="0.2" ray_count="5" />
   <!-- rear sensor -->
-  <xacro:urm04_sensor frame_name="rear_range" ros_topic="rear_range" update_rate="10" min_range="0.01" max_range="2" horizontal_field_of_view="0.261799" vertical_field_of_view="0.2" ray_count="2" />
+  <xacro:urm04_sensor frame_name="rear_range" ros_topic="rear_range" update_rate="10" min_range="0.01" max_range="2" horizontal_field_of_view="0.261799" vertical_field_of_view="0.2" ray_count="5" />
+  <xacro:urm04_sensor frame_name="front_right_range" ros_topic="front_right_range" update_rate="10" min_range="0.01" max_range="2" horizontal_field_of_view="0.261799" vertical_field_of_view="0.2" ray_count="5" />
+  <xacro:urm04_sensor frame_name="front_left_range" ros_topic="front_left_range" update_rate="10" min_range="0.01" max_range="2" horizontal_field_of_view="0.261799" vertical_field_of_view="0.2" ray_count="5" />
+  <xacro:urm04_sensor frame_name="rear_right_range" ros_topic="rear_right_range" update_rate="10" min_range="0.01" max_range="2" horizontal_field_of_view="0.261799" vertical_field_of_view="0.2" ray_count="5" />
+  <xacro:urm04_sensor frame_name="rear_left_range" ros_topic="rear_left_range" update_rate="10" min_range="0.01" max_range="2" horizontal_field_of_view="0.261799" vertical_field_of_view="0.2" ray_count="5" />
 </robot>

Commit message: Update sim to include RPLidar A2

File: nexus_4wd_mecanum_description/urdf/nexus_4wd_mecanum.xacro (robot description, xacro)
@@ -270,5 +270,5 @@
     </inertial>
   </link>
-  <joint name="left_sensor_joint" type="fixed">
+  <!-- <joint name="left_sensor_joint" type="fixed">
     <origin xyz="0 0.108 0.010" rpy="0 -0.1 ${PI/2}" />
     <parent link="base_link"/>
@@ -381,4 +381,31 @@
       <material name="black" />
     </visual>
+  </link> -->
+  <joint name="rplidar_joint" type="fixed">
+    <axis xyz="0 1 0" />
+    <origin xyz="0.02 0 0.058" rpy="0 0 3.14"/>
+    <parent link="base_link"/>
+    <child link="laser"/>
+  </joint>
+  <!-- rplidar Laser -->
+  <link name="laser">
+    <!-- <collision>
+      <origin xyz="0 0 0" rpy="1.5707 0 4.71"/>
+      <geometry>
+        <mesh filename="package://rosbot_description/meshes/rplidar.stl" scale="0.001 0.001 0.001" />
+      </geometry>
+    </collision>
+    <visual>
+      <origin xyz="0 0 0" rpy="1.5707 0 4.71"/>
+      <geometry>
+        <mesh filename="package://rosbot_description/meshes/rplidar.stl" scale="0.001 0.001 0.001" />
+      </geometry>
+      <material name="Black"/>
+    </visual> -->
+    <inertial>
+      <mass value="1e-5" />
+      <origin xyz="0 0 0" rpy="1.5707 0 4.71"/>
+      <inertia ixx="0" ixy="0" ixz="0" iyy="0" iyz="0" izz="0" />
+    </inertial>
   </link>
   <!-- Include controller plugin for Gazebo -->
@@ -387,14 +414,14 @@
   <xacro:include filename="$(find nexus_4wd_mecanum_description)/urdf/urm04_sensor.xacro"/>
   <!-- front sensor -->
-  <xacro:urm04_sensor frame_name="front_range" ros_topic="front_range" update_rate="10" min_range="0.01" max_range="2" horizontal_field_of_view="0.261799" vertical_field_of_view="0.2" ray_count="5" />
+  <xacro:urm04_sensor frame_name="front_range" ros_topic="range/front_forward" update_rate="10" min_range="0.01" max_range="2" horizontal_field_of_view="0.261799" vertical_field_of_view="0.2" ray_count="5" />
   <!-- left sensor -->
-  <xacro:urm04_sensor frame_name="left_range" ros_topic="left_range" update_rate="10" min_range="0.01" max_range="2" horizontal_field_of_view="0.261799" vertical_field_of_view="0.2" ray_count="5" />
+  <xacro:urm04_sensor frame_name="left_range" ros_topic="range/left" update_rate="10" min_range="0.01" max_range="2" horizontal_field_of_view="0.261799" vertical_field_of_view="0.2" ray_count="5" />
   <!-- right sensor -->
-  <xacro:urm04_sensor frame_name="right_range" ros_topic="right_range" update_rate="10" min_range="0.01" max_range="2" horizontal_field_of_view="0.261799" vertical_field_of_view="0.2" ray_count="5" />
+  <xacro:urm04_sensor frame_name="right_range" ros_topic="range/right" update_rate="10" min_range="0.01" max_range="2" horizontal_field_of_view="0.261799" vertical_field_of_view="0.2" ray_count="5" />
   <!-- rear sensor -->
-  <xacro:urm04_sensor frame_name="rear_range" ros_topic="rear_range" update_rate="10" min_range="0.01" max_range="2" horizontal_field_of_view="0.261799" vertical_field_of_view="0.2" ray_count="5" />
-  <xacro:urm04_sensor frame_name="front_right_range" ros_topic="front_right_range" update_rate="10" min_range="0.01" max_range="2" horizontal_field_of_view="0.261799" vertical_field_of_view="0.2" ray_count="5" />
-  <xacro:urm04_sensor frame_name="front_left_range" ros_topic="front_left_range" update_rate="10" min_range="0.01" max_range="2" horizontal_field_of_view="0.261799" vertical_field_of_view="0.2" ray_count="5" />
-  <xacro:urm04_sensor frame_name="rear_right_range" ros_topic="rear_right_range" update_rate="10" min_range="0.01" max_range="2" horizontal_field_of_view="0.261799" vertical_field_of_view="0.2" ray_count="5" />
-  <xacro:urm04_sensor frame_name="rear_left_range" ros_topic="rear_left_range" update_rate="10" min_range="0.01" max_range="2" horizontal_field_of_view="0.261799" vertical_field_of_view="0.2" ray_count="5" />
+  <xacro:urm04_sensor frame_name="rear_range" ros_topic="range/rear" update_rate="10" min_range="0.01" max_range="2" horizontal_field_of_view="0.261799" vertical_field_of_view="0.2" ray_count="5" />
+  <xacro:urm04_sensor frame_name="front_right_range" ros_topic="range/front_right" update_rate="10" min_range="0.01" max_range="2" horizontal_field_of_view="0.261799" vertical_field_of_view="0.2" ray_count="5" />
+  <xacro:urm04_sensor frame_name="front_left_range" ros_topic="range/front_left" update_rate="10" min_range="0.01" max_range="2" horizontal_field_of_view="0.261799" vertical_field_of_view="0.2" ray_count="5" />
+  <xacro:urm04_sensor frame_name="rear_right_range" ros_topic="range/rear_right" update_rate="10" min_range="0.01" max_range="2" horizontal_field_of_view="0.261799" vertical_field_of_view="0.2" ray_count="5" />
+  <xacro:urm04_sensor frame_name="rear_left_range" ros_topic="range/rear_left" update_rate="10" min_range="0.01" max_range="2" horizontal_field_of_view="0.261799" vertical_field_of_view="0.2" ray_count="5" />
 </robot>
